Commit message: dw_simulation pkg

File: src/boxbot_description/urdf/box_bot3.gazebo.xacro (robot description, xacro)
@@ -1,9 +1,63 @@
 <?xml version="1.0"?>
 <robot xmlns:xacro="http://www.ros.org/wiki/xacro">
+    <gazebo>
+        <plugin name="joint_state_publisher" filename="libgazebo_ros_joint_state_publisher.so">
+            <ros>
+                <remapping>~/out:=joint_states</remapping>
+            </ros>
+            <update_rate>50</update_rate>
+            <joint_name>left_wheel_joint</joint_name>
+            <joint_name>right_wheel_joint</joint_name>
+        </plugin>
+    </gazebo>
+    <gazebo>
+        <plugin name="differential_drive_controller" filename="libgazebo_ros_diff_drive.so">
+            <ros>
+                <namespace>/</namespace>
+                <remapping>cmd_vel:=cmd_vel</remapping>
+                <remapping>odom:=odom</remapping>
+            </ros>
+            <update_rate>50</update_rate>
+            <left_joint>left_wheel_joint</left_joint>
+            <right_joint>right_wheel_joint</right_joint>
+            <wheel_separation>0.12</wheel_separation>
+            <wheel_diameter>0.07</wheel_diameter>
+            <!-- <max_wheel_torque>5.0</max_wheel_torque>
+            <max_wheel_acceleration>0.5</max_wheel_acceleration> -->
+            <max_wheel_torque>100</max_wheel_torque>
+            <max_wheel_acceleration>0.7</max_wheel_acceleration>
+            <publish_odom>true</publish_odom>
+            <publish_odom_tf>false</publish_odom_tf>
+            <publish_wheel_tf>false</publish_wheel_tf>
+            <odometry_frame>odom</odometry_frame>
+            <robot_base_frame>base_footprint</robot_base_frame>
+            <covariance_x>0.05</covariance_x>
+            <covariance_y>0.05</covariance_y>
+            <covariance_yaw>0.1</covariance_yaw>
+<!--
+            <publish_odom>true</publish_odom>
+            <publish_odom_tf>false</publish_odom_tf>
+            <publish_wheel_tf>false</publish_wheel_tf>
+            <odometry_frame>odom</odometry_frame>
+            <robot_base_frame>base_footprint</robot_base_frame>
+            <covariance_x>0.001</covariance_x>
+            <covariance_y>0.001</covariance_y>
+            <covariance_yaw>0.01</covariance_yaw> -->
+        </plugin>
+    </gazebo>
     <gazebo reference="camera_link">
+        <visual>
+            <material>
+                <ambient>0.3 0.3 0.3 1.0</ambient>
+                <diffuse>0.3 0.3 0.3 1.0</diffuse>
+                <specular>0.01 0.01 0.01 1.0</specular>
+                <emissive>0.0 0.0 0.0 1.0</emissive>
+            </material>
+        </visual>
         <sensor name="camera" type="depth">
+            <always_on>true</always_on>
             <visualize>true</visualize>
-            <update_rate>30.0</update_rate>
-            <camera name="camera">
+            <update_rate>15.0</update_rate>
+            <camera name="d435i">
                 <horizontal_fov>1.5184</horizontal_fov>
                 <image>
@@ -13,5 +67,5 @@
                 </image>
                 <clip>
-                    <near>0.1</near>
+                    <near>0.105</near>
                     <far>10.0</far>
                 </clip>
@@ -20,40 +74,52 @@
                 <ros>
                     <namespace>camera</namespace>
-                    <remapping>camera/image_raw:=color/image_raw</remapping>
-                    <remapping>camera/depth/image_raw:=depth/image_rect_raw</remapping>
-                    <remapping>camera/camera_info:=color/camera_info</remapping>
-                    <remapping>camera/depth/camera_info:=depth/camera_info</remapping>
-                    <remapping>camera/points:=depth/color/points</remapping>
+                    <remapping>d435i/image_raw:=color/image_raw</remapping>
+                    <remapping>d435i/camera_info:=color/camera_info</remapping>
+                    <remapping>d435i/depth/image_raw:=depth/image_rect_raw</remapping>
+                    <remapping>d435i/depth/camera_info:=depth/camera_info</remapping>
+                    <remapping>d435i/points:=depth/color/points</remapping>
                 </ros>
                 <camera_name>d435i</camera_name>
-                <frame_name>camera_depth_optical_frame</frame_name> <hack_baseline>0.07</hack_baseline>
-                <min_depth>0.1</min_depth>
-                <max_depth>5.0</max_depth>
+                <frame_name>camera_depth_optical_frame</frame_name>
+                <hack_baseline>0.05</hack_baseline>
+                <min_depth>0.105</min_depth>
+                <max_depth>10.0</max_depth>
             </plugin>
         </sensor>
     </gazebo>
-    <gazebo>
-        <plugin name="joint_state_publisher" filename="libgazebo_ros_joint_state_publisher.so">
-            <ros>
-                <remapping>~/out:=joint_states</remapping>
-            </ros>
-            <update_rate>30</update_rate>
-            <joint_name>left_wheel_joint</joint_name>
-            <joint_name>right_wheel_joint</joint_name>
-        </plugin>
-    </gazebo>
-    <gazebo>
-        <plugin name="differential_drive_controller" filename="libgazebo_ros_diff_drive.so">
-            <left_joint>left_wheel_joint</left_joint>
-            <right_joint>right_wheel_joint</right_joint>
-            <wheel_separation>${wheel_ygap * 2}</wheel_separation>
-            <wheel_diameter>${wheel_radius * 2}</wheel_diameter>
-            <max_wheel_torque>1.0</max_wheel_torque>
-            <max_wheel_acceleration>2.0</max_wheel_acceleration>
-            <publish_odom>true</publish_odom>
-            <publish_odom_tf>true</publish_odom_tf>
-            <odometry_frame>odom</odometry_frame>
-            <robot_base_frame>base_footprint</robot_base_frame>
-        </plugin>
+    <gazebo reference="laser_scan_link">
+        <sensor name="lidar_sensor" type="ray">
+            <always_on>true</always_on>
+            <visualize>true</visualize>
+            <update_rate>10</update_rate>
+            <ray>
+                <scan>
+                    <horizontal>
+                        <samples>360</samples>
+                        <resolution>1.0</resolution>
+                        <min_angle>-3.14159</min_angle>
+                        <max_angle>3.14159</max_angle>
+                    </horizontal>
+                </scan>
+                <range>
+                    <min>0.12</min>
+                    <max>8.0</max>
+                    <resolution>0.01</resolution>
+                </range>
+                <noise>
+                    <type>gaussian</type>
+                    <mean>0.0</mean>
+                    <stddev>0.01</stddev>
+                </noise>
+            </ray>
+            <plugin name="scan_controller" filename="libgazebo_ros_ray_sensor.so">
+                <ros>
+                    <remapping>~/out:=scan</remapping>
+                    <use_sim_time>true</use_sim_time>
+                </ros>
+                <output_type>sensor_msgs/LaserScan</output_type>
+                <frame_name>laser_scan_link</frame_name>
+            </plugin>
+        </sensor>
     </gazebo>
     <gazebo reference="imu_link">
@@ -79,33 +145,5 @@
                 </ros>
                 <initial_orientation_as_reference>false</initial_orientation_as_reference>
-            </plugin>
-        </sensor>
-    </gazebo>
-    <gazebo reference="laser_scan_link">
-        <sensor name="lidar" type="ray">
-            <always_on>true</always_on>
-            <visualize>true</visualize>
-            <update_rate>10</update_rate>
-            <ray>
-                <scan>
-                    <horizontal>
-                        <samples>360</samples>
-                        <resolution>1.0</resolution>
-                        <min_angle>0.00</min_angle>
-                        <max_angle>6.28</max_angle>
-                    </horizontal>
-                </scan>
-                <range>
-                    <min>0.12</min>
-                    <max>12.0</max>
-                    <resolution>0.015</resolution>
-                </range>
-            </ray>
-            <plugin name="scan_controller" filename="libgazebo_ros_ray_sensor.so">
-                <ros>
-                    <remapping>~/out:=scan</remapping>
-                </ros>
-                <output_type>sensor_msgs/LaserScan</output_type>
-                <frame_name>laser_scan_link</frame_name>
+                <gaussianNoise>0.01</gaussianNoise>
             </plugin>
         </sensor>

File: src/boxbot_description/urdf/box_bot3.urdf.xacro (robot description, xacro)
@@ -1,16 +1,16 @@
 <?xml version="1.0"?>
 <robot xmlns:xacro="http://www.ros.org/wiki/xacro" name="box_bot">
-    <xacro:property name="base_mass"   value="0.8"/>
+    <xacro:property name="base_mass"   value="2.0"/>
     <xacro:property name="base_size"   value="0.1"/>
     <xacro:property name="ground_clearance" value="0.01"/>
-    <xacro:property name="wheel_mass"  value="0.05"/>
+    <xacro:property name="wheel_mass"  value="0.2"/>
     <xacro:property name="wheel_radius" value="0.035"/>
     <xacro:property name="wheel_length" value="0.01"/>
-    <xacro:property name="wheel_ygap"   value="0.05"/>
-    <xacro:property name="caster_mass"   value="0.01"/>
+    <xacro:property name="wheel_ygap"   value="0.06"/>
+    <xacro:property name="caster_mass"   value="0.1"/>
     <xacro:property name="caster_radius" value="0.01"/>
     <xacro:property name="caster_xgap"   value="0.035"/>
     <xacro:include filename="box_bot3.gazebo.xacro" />
-    <xacro:include filename="$(find realsense2_description)/urdf/_d435i.urdf.xacro" />
+    <xacro:include filename="$(find realsense2_description)/urdf/_d435i.urdf.xacro"/>
     <material name="red"><color rgba="1.0 0.0 0.0 1"/></material>
     <material name="green_dark"><color rgba="0.0 0.5 0.0 1"/></material>
@@ -26,33 +26,33 @@
         </visual>
         <collision>
+            <origin xyz="0 0 0.005" rpy="0 0 0"/>
             <geometry>
-                <box size="${base_size} ${base_size} ${base_size}"/>
+                <box size="${base_size} ${base_size} 0.08"/>
             </geometry>
         </collision>
         <inertial>
             <mass value="${base_mass}"/>
-            <origin rpy="0 0 0" xyz="0 0 -0.02"/>
-            <inertia ixx="0.001333" ixy="0" ixz="0" iyy="0.001333" iyz="0" izz="0.001333"/>
-        </inertial>
+            <origin xyz="0.01 0 0" rpy="0 0 0"/>
+            <inertia ixx="0.00227" ixy="0" ixz="0" iyy="0.00227" iyz="0" izz="0.00333"/> </inertial>
     </link>
     <joint name="base_link_joint" type="fixed">
-        <origin xyz="0 0 ${ground_clearance + (base_size/2)}" rpy="0 0 0"/>
+        <origin xyz="0 0 0.06" rpy="0 0 0"/>
         <parent link="base_footprint" />
         <child link="base_link" />
     </joint>
     <xacro:sensor_d435i parent="base_link" name="camera" use_nominal_extrinsics="true">
-    <origin xyz="0.06 0 0.025" rpy="0 -0.2 0"/>
+        <origin xyz="0.053 0 0.05" rpy="0 0 0"/>
     </xacro:sensor_d435i>
     <xacro:macro name="wheel" params="prefix side color">
         <link name="${prefix}_wheel_link">
             <visual>
-                <origin xyz="0 ${side * 0.005} 0" rpy="0 1.5707 1.5707"/>
+                <origin xyz="0 0 0" rpy="1.5707 0 0"/>
                 <geometry>
                     <cylinder length="${wheel_length}" radius="${wheel_radius}"/>
                 </geometry>
-                <material name="black"/>
+                <material name="orange"/>
             </visual>
             <collision>
-                <origin xyz="0 ${side * 0.005} 0" rpy="0 1.5707 1.5707"/>
+                <origin xyz="0 0 0" rpy="1.5707 0 0"/>
                 <geometry>
                     <cylinder length="${wheel_length}" radius="${wheel_radius}"/>
@@ -60,7 +60,7 @@
             </collision>
             <inertial>
-                <origin xyz="0 ${side * 0.005} 0" rpy="0 1.5707 1.5707"/>
+                <origin xyz="0 0 0" rpy="1.5707 0 0"/>
                 <mass value="${wheel_mass}"/>
-                <inertia ixx="1.5316e-05" ixy="0" ixz="0" iyy="1.5316e-05" iyz="0" izz="3.0625e-05"/>
+                <inertia ixx="0.000063" ixy="0" ixz="0" iyy="0.0001225" iyz="0" izz="0.000063"/>
             </inertial>
         </link>
@@ -71,11 +71,13 @@
             <axis xyz="0 1 0"/>
             <limit effort="10.0" velocity="10.0"/>
-            <dynamics damping="0.1" friction="0.1"/>
+            <dynamics damping="1.0" friction="1.0"/>
         </joint>
         <gazebo reference="${prefix}_wheel_link">
-            <kp>1000000.0</kp>
-            <kd>10.0</kd>
             <mu1>10.0</mu1>
             <mu2>10.0</mu2>
+            <kp>1000000.0</kp>
+            <kd>100.0</kd>
+            <minDepth>0.001</minDepth>
+            <maxVel>0.1</maxVel>
             <fdir1>1 0 0</fdir1>
             <material>Gazebo/${color}</material>
@@ -83,5 +85,5 @@
     </xacro:macro>
     <xacro:wheel prefix="left"  side="1"  color="Green"/>
-    <xacro:wheel prefix="right" side="-1" color="Green"/>
+    <xacro:wheel prefix="right" side="-1" color="Orange"/>
     <xacro:macro name="caster" params="prefix x_pos">
         <link name="${prefix}_caster_link">
@@ -95,5 +97,5 @@
             <inertial>
                 <mass value="${caster_mass}"/>
-                <inertia ixx="4e-07" ixy="0" ixz="0" iyy="4e-07" iyz="0" izz="4e-07"/>
+                <inertia ixx="0.000004" ixy="0" ixz="0" iyy="0.000004" iyz="0" izz="0.000004"/>
             </inertial>
         </link>
@@ -104,6 +106,11 @@
         </joint>
         <gazebo reference="${prefix}_caster_link">
-            <mu1>0.01</mu1>
-            <mu2>0.01</mu2>
+            <mu1>0.0</mu1>
+            <mu2>0.0</mu2>
+            <slip1>1.0</slip1>
+            <slip2>1.0</slip2>
+            <kp>1000000.0</kp>
+            <kd>100.0</kd>
+            <minDepth>0.001</minDepth>
             <material>Gazebo/Purple</material>
         </gazebo>
@@ -111,42 +118,35 @@
     <xacro:caster prefix="front" x_pos="${caster_xgap}"/>
     <xacro:caster prefix="back"  x_pos="${-caster_xgap}"/>
-    <!-- Laser Position Control -->
     <link name="laser_scan_link">
         <visual>
             <origin xyz="0 0 0" rpy="0 0 0" />
-            <geometry>
-                <mesh filename="package://boxbot_description/meshes/sensors/rplidar.dae" scale="1.0 1.0 1.0"/>
-            </geometry>
+            <geometry><mesh filename="package://boxbot_description/meshes/sensors/rplidar.dae" scale="1.0 1.0 1.0"/></geometry>
         </visual>
         <collision>
             <origin xyz="0 0 0.0204" rpy="0 0 0"/>
-            <geometry>
-                <cylinder length="0.0408" radius="0.037493"/>
-            </geometry>
+            <geometry><cylinder length="0.0408" radius="0.0375"/></geometry>
         </collision>
         <inertial>
             <mass value="0.01"/>
             <origin xyz="0 0 0.0204" rpy="0 0 0"/>
-            <inertia ixx="6.066578520833334e-06" ixy="0" ixz="0" iyy="6.072950163333333e-06" iyz="0" izz="9.365128684166666e-06"/>
+            <inertia ixx="6.06e-06" ixy="0" ixz="0" iyy="6.07e-06" iyz="0" izz="9.36e-06"/>
         </inertial>
     </link>
-    <!-- <joint name="laser_scan_link_joint" type="continuous"> -->
     <joint name="laser_scan_link_joint" type="fixed">
         <origin rpy="0 0 0" xyz="0 0 0.05"/>
         <parent link="base_link"/>
         <child link="laser_scan_link"/>
-        <!-- <axis xyz="0 0 1"/>
-        <limit effort="10.0" velocity="100.0"/>
-        <dynamics damping="0.01" friction="0.01"/> -->
     </joint>
-    <!-- IMU -->
     <link name="imu_link">
         <visual>
             <origin xyz="0 0 0" rpy="0 0 0"/>
-            <geometry>
-                <box size="0.015 0.015 0.0025"/>
-            </geometry>
+            <geometry><box size="0.015 0.015 0.0025"/></geometry>
             <material name="blue"/>
         </visual>
+        <inertial>
+            <mass value="0.001"/>
+            <origin xyz="0 0 0" rpy="0 0 0"/>
+            <inertia ixx="0.000001" ixy="0" ixz="0" iyy="0.000001" iyz="0" izz="0.000001"/>
+        </inertial>
     </link>
     <joint name="imu_joint" type="fixed">
@@ -155,3 +155,6 @@
         <child link="imu_link"/>
     </joint>
-    </robot>
+    <gazebo reference="imu_link">
+        <material>Gazebo/Red</material>
+    </gazebo>
+</robot>
