Commit message: add(5/4) ros2_control 관련 설정 및 시뮬레이션용 런치 파일 추가, SLAM과 localization 런치 파일에서 시뮬레이션 타임 사용하도록 수정

File: src/tb3_description/urdf/tb3_burger_gazebo_ros2_control.xacro (robot description, xacro)
@@ -79,4 +79,5 @@
     <!-- <material>Gazebo/FlatBlack</material> -->
   </gazebo>
+<!--
   <gazebo>
     <plugin name="tb3_diff_drive" filename="libgazebo_ros_diff_drive.so">
@@ -103,4 +104,36 @@
       <joint_name>wheel_left_joint</joint_name>
       <joint_name>wheel_right_joint</joint_name>
+    </plugin>
+  </gazebo> -->
+  <ros2_control name="GazeboSystem" type="system">
+    <hardware>
+      <plugin>gazebo_ros2_control/GazeboSystem</plugin>
+    </hardware>
+    <joint name="wheel_left_joint">
+      <command_interface name="velocity">
+        <param name="min">-10</param>
+        <param name="max">10</param>
+      </command_interface>
+      <state_interface name="position"/>
+      <state_interface name="velocity"/>
+    </joint>
+    <joint name="wheel_right_joint">
+      <command_interface name="velocity">
+        <param name="min">-10</param>
+        <param name="max">10</param>
+      </command_interface>
+      <state_interface name="position"/>
+      <state_interface name="velocity"/>
+    </joint>
+  </ros2_control>
+  <gazebo>
+    <plugin name="gazebo_ros2_control" filename="libgazebo_ros2_control.so">
+      <!-- <parameters>$(find boxbot_bringup)/config/controllers.yaml</parameters> -->
+      <parameters>$(find boxbot_bringup)/config/controllers_advenced.yaml</parameters>
+      <ros>
+        <use_sim_time>true</use_sim_time>
+        <remapping>/diff_drive_controller/cmd_vel_unstamped:=/cmd_vel</remapping>
+        <!-- <remapping>/diff_drive_controller/odom:=/odom</remapping> -->
+      </ros>
     </plugin>
   </gazebo>
@@ -156,4 +189,5 @@
       <plugin name="tb3_imu" filename="libgazebo_ros_imu_sensor.so">
         <ros><remapping>~/out:=imu</remapping></ros>
+        <frame_name>imu_link</frame_name>
         <gaussianNoise>0.01</gaussianNoise>
       </plugin>

File: src/tb3_description/urdf/tb3_burger_main.urdf.xacro (robot description, xacro)
@@ -4,5 +4,5 @@
   vlp16
   lds -->
-  <xacro:arg name="lidar_model" default="vlp16"/> <xacro:property name="lidar_selection" value="$(arg lidar_model)" />
+  <xacro:arg name="lidar_model" default="lds"/> <xacro:property name="lidar_selection" value="$(arg lidar_model)" />
   <xacro:property name="wheel_width"  value="0.018" />
   <xacro:property name="wheel_radius" value="0.033" />
@@ -13,5 +13,6 @@
   <!-- <xacro:include filename="$(find tb3_description)/urdf/common_properties.xacro"/> -->
   <xacro:include filename="$(find tb3_description)/urdf/xkcd_colors.urdf.xacro"/>
-  <xacro:include filename="$(find tb3_description)/urdf/tb3_burger_gazebo.xacro"/>
+  <!-- <xacro:include filename="$(find tb3_description)/urdf/tb3_burger_gazebo.xacro"/>  -->
+  <xacro:include filename="$(find tb3_description)/urdf/tb3_burger_gazebo_ros2_control.xacro"/>
   <xacro:include filename="$(find realsense2_description)/urdf/_d435i.urdf.xacro"/>
   <xacro:include filename="$(find tb3_description)/urdf/VLP16.urdf.xacro"/>
